File: KDT_Hierarchical_KiBot.kicad_pcb (KiCad board)
At the start: 6 copper layers, 0 parts

Commit message: [Added] Some dumy circuit
Parts:
- added C1: 47uF, Capacitor_SMD:CP_Elec_8x10, F.Cu at (125.3, 100.6)
- added C2: 100nF, Capacitor_SMD:C_0805_2012Metric, F.Cu at (117.5, 96.6)
- added C3: 22pF, Capacitor_SMD:C_0805_2012Metric, F.Cu at (156.7, 80.8)
- added C4: 22pF, Capacitor_SMD:C_0805_2012Metric, F.Cu at (150.4, 80.8)
- added C5: 1uF, Capacitor_SMD:C_0805_2012Metric, F.Cu at (157.8, 94.8)
- added C6: 100nF, Capacitor_SMD:C_0805_2012Metric, F.Cu at (156.9, 87.8)
- added C7: 100nF, Capacitor_SMD:C_0805_2012Metric, F.Cu at (148.4, 84.6)
- added C8: 100nF, Capacitor_SMD:C_0805_2012Metric, F.Cu at (139.2, 84.7)
- added D1: CD1206-S01575, Diode_SMD:D_1206_3216Metric, F.Cu at (157.3, 102.5)
- added D2: LED, LED_SMD:LED_0805_2012Metric, F.Cu at (141.8, 80.6)
- added D3: LED, LED_SMD:LED_0805_2012Metric, F.Cu at (139.3, 80.6)
- added F1: MF-MSMF050-2, Resistor_SMD:R_1812_4532Metric, F.Cu at (162.4, 82.9)
- added FB1: BLM21PG221SN1D, Resistor_SMD:R_0805_2012Metric, F.Cu at (162.4, 96.4)
- added FID1: Fiducial, Fiducial:Fiducial_0.75mm_Mask1.5mm, F.Cu at (163.9, 76.3)
- added FID2: Fiducial, Fiducial:Fiducial_0.75mm_Mask1.5mm, F.Cu at (166.2, 103.0)
- added FID3: Fiducial, Fiducial:Fiducial_0.75mm_Mask1.5mm, F.Cu at (124.5, 75.8)
- added FID4: Fiducial, Fiducial:Fiducial_0.75mm_Mask1.5mm, F.Cu at (131.7, 103.9)
- added H1: MountingHole, MountingHole:MountingHole_2.7mm_M2.5, F.Cu at (171.5, 102.7)
- added H2: MountingHole, MountingHole:MountingHole_2.7mm_M2.5, F.Cu at (117.5, 102.7)
- added H3: MountingHole, MountingHole:MountingHole_2.7mm_M2.5, F.Cu at (117.5, 75.2)
- added H4: MountingHole, MountingHole:MountingHole_2.7mm_M2.5, F.Cu at (171.5, 75.2)
- added J1: Barrel_Jack_Switch, Connector_BarrelJack:BarrelJack_CLIFF_FC681465S_SMT_Horizontal, F.Cu at (120.6, 86.9)
- added J2: USB_B, Connector_USB:USB_B_Lumberg_2411_02_Horizontal, F.Cu at (168.0, 87.2)
- added J3: P1, Connector_PinHeader_2.54mm:PinHeader_1x05_P2.54mm_Vertical, F.Cu at (130.8, 85.2)
- added J4: 2x2M, Connector_PinHeader_2.54mm:PinHeader_2x02_P2.54mm_Vertical, F.Cu at (146.4, 100.9)
- added J5: ICSP1, Connector_PinHeader_2.54mm:PinHeader_2x03_P2.54mm_Vertical, F.Cu at (135.6, 103.5)
- added J6: P2, Connector_PinHeader_2.54mm:PinHeader_1x06_P2.54mm_Vertical, F.Cu at (135.4, 82.9)
- added JP1: SolderJumper_2_Open, Jumper:SolderJumper-2_P1.3mm_Open_RoundedPad1.0x1.5mm, F.Cu at (161.7, 101.5)
- added R1: 22R, Resistor_SMD:R_0805_2012Metric, F.Cu at (160.8, 91.8)
- added R2: 22R, Resistor_SMD:R_0805_2012Metric, F.Cu at (160.8, 89.5)
- added R3: 1M, Resistor_SMD:R_0805_2012Metric, F.Cu at (153.4, 81.6)
- added R4: 10K, Resistor_SMD:R_0805_2012Metric, F.Cu at (153.5, 101.5)
- added R5: 1K, Resistor_SMD:R_0805_2012Metric, F.Cu at (139.2, 88.5)
- added R6: 1K, Resistor_SMD:R_0805_2012Metric, F.Cu at (141.8, 75.9)
- added R7: 1K, Resistor_SMD:R_0805_2012Metric, F.Cu at (139.3, 75.9)
- added TP2: TestPoint, TestPoint:TestPoint_Pad_D1.0mm, B.Cu at (162.3, 85.9)
- added TP3: TestPoint, TestPoint:TestPoint_Pad_D1.0mm, B.Cu at (168.0, 84.2)
- added TP4: TestPoint, TestPoint:TestPoint_Pad_D1.0mm, B.Cu at (173.5, 86.5)
- added TP5: TestPoint, TestPoint:TestPoint_Pad_D1.0mm, B.Cu at (173.5, 89.8)
- added TP6: TestPoint, TestPoint:TestPoint_Pad_D1.0mm, B.Cu at (158.8, 75.7)
- added TP8: TestPoint, TestPoint:TestPoint_Pad_D1.0mm, B.Cu at (148.0, 75.7)
- added TP9: TestPoint, TestPoint:TestPoint_Pad_D1.0mm, B.Cu at (150.4, 90.3)
- added U1: ATmega8U2-AU, Package_QFP:TQFP-32_7x7mm_P0.8mm, F.Cu at (148.9, 91.5)
- added VR1: CG0603MLC-05E, Resistor_SMD:R_0603_1608Metric, F.Cu at (164.9, 93.0)
- added VR2: CG0603MLC-05E, Resistor_SMD:R_0603_1608Metric, F.Cu at (164.9, 88.0)
- added Y1: 16MHz, Crystal:Crystal_SMD_Abracon_ABM3-2Pin_5.0x3.2mm, F.Cu at (153.4, 75.7)
Routing:
- net Earth: track 0.00 -> 49.0 mm, vias 0 -> 5
- net Net-(J2-Shield): track 0.00 -> 39.3 mm, vias 0 -> 3
- net Net-(J3-Pin_1): track 0.00 -> 36.5 mm, vias 0 -> 1
- net Net-(J3-Pin_2): track 0.00 -> 35.6 mm, vias 0 -> 1
- net Net-(J3-Pin_4): track 0.00 -> 33.5 mm, vias 0 -> 1
- net Net-(J3-Pin_3): track 0.00 -> 32.6 mm, vias 0 -> 1
- net Net-(J3-Pin_5): track 0.00 -> 30.8 mm
- net +5V: track 0.00 -> 30.5 mm, vias 0 -> 8
- net /RESET2: track 0.00 -> 28.5 mm
- net GND: track 0.00 -> 24.5 mm, vias 0 -> 11
- net Net-(J6-Pin_6): track 0.00 -> 19.3 mm, vias 0 -> 1
- net Net-(U1-XTAL1): track 0.00 -> 18.9 mm, vias 0 -> 1
- net Net-(U1-PC0/XTAL2): track 0.00 -> 18.3 mm, vias 0 -> 1
- net /MISO2: track 0.00 -> 18.0 mm
- net Net-(J6-Pin_5): track 0.00 -> 16.9 mm, vias 0 -> 1
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- added copper zone on In1.Cu, net Earth
- added copper zone on In1.Cu, net GND
- added copper zone on In1.Cu, net Net-(J2-Shield)
