File: KDT_Hierarchical_KiBot.kicad_pcb (KiCad board)
At the start: 6 copper layers, 46 parts, among them J1 Barrel_Jack_Switch, J2 USB_B, J3 P1, J4 2x2M, J5 ICSP1, J6 P2, U1 ATmega8U2-AU, Y1 16MHz

Commit message: [Added] Edege cuts
Other:
- board outline added: 63.2 x 35.8 mm
- board text added: "0.02mm"
- board text added: "0.035mm (1.00oz)"
- board text added: "0.07mm (2.00oz)"
- board text added: "0.18mm"
- board text added: "0.4mm"
- board text added: "B.Mask"
- board text added: "B.Paste"
- board text added: "B.Silkscreen"
- board text added: "Copper"
- board text added: "Core"
- board text added: "Dielectric"
- board text added: "Direct Printing"
- board text added: "F.Mask"
- board text added: "F.Paste"
- board text added: "F.Silkscreen"
- board text added: "FR4"
- board text added: "FR4_7628"
- board text added: "GBR"
- board text added: "Gerber"
- board text added: "L1 (Sig, PWR)"
- board text added: "L2 (GND)"
- board text added: "L3 (Sig, PWR)"
- board text added: "L4 (Sig, PWR)"
- board text added: "L5 (GND)"
- board text added: "L6 (Sig, PWR)"
- board text added: "Layer"
- board text added: "Legend"
- board text added: "Material"
- board text added: "Note: external layer thicknesses are specified after plating"
- board text added: "Paste Mask"
- board text added: "Plane"
- board text added: "Prepreg"
- board text added: "Signal"
- board text added: "Solder Mask"
- board text added: "Solder Resist"
- board text added: "Thickness"
- board text added: "Total thickness: 1.66mm"
- board text added: "Type"
