File: Section A - Title A.kicad_sch (KiCad schematic)
At the start: 0 parts

Commit message: [Added] Some dumy circuit
Parts:
- added C1: 47uF, Capacitor_SMD:CP_Elec_8x10, symbol Device:C_Polarized
- added C2, C6, C7, C8: 100nF, Capacitor_SMD:C_0805_2012Metric, symbol Device:C
- added C3, C4: 22pF, Capacitor_SMD:C_0805_2012Metric, symbol Device:C
- added C5: 1uF, Capacitor_SMD:C_0805_2012Metric, symbol Device:C
- added D1: CD1206-S01575, Diode_SMD:D_1206_3216Metric, symbol Device:D
- added D2, D3: LED, LED_SMD:LED_0805_2012Metric, symbol Device:LED
- added F1: MF-MSMF050-2, Resistor_SMD:R_1812_4532Metric, symbol Device:Polyfuse
- added FB1: BLM21PG221SN1D, Resistor_SMD:R_0805_2012Metric, symbol Device:FerriteBead
- added FID1, FID2, FID3, FID4: Fiducial, Fiducial:Fiducial_0.75mm_Mask1.5mm, symbol Mechanical:Fiducial
- added H1, H2, H3, H4: MountingHole, MountingHole:MountingHole_2.7mm_M2.5, symbol Mechanical:MountingHole
- added J1: Barrel_Jack_Switch, Connector_BarrelJack:BarrelJack_CLIFF_FC681465S_SMT_Horizontal, symbol Connector:Barrel_Jack_Switch
- added J2: USB_B, Connector_USB:USB_B_Lumberg_2411_02_Horizontal, symbol Connector:USB_B
- added J3: P1, Connector_PinHeader_2.54mm:PinHeader_1x05_P2.54mm_Vertical, symbol Connector:Conn_01x05_Pin
- added J4: 2x2M, Connector_PinHeader_2.54mm:PinHeader_2x02_P2.54mm_Vertical, symbol Connector_Generic:Conn_02x02_Odd_Even
- added J5: ICSP1, Connector_PinHeader_2.54mm:PinHeader_2x03_P2.54mm_Vertical, symbol Connector_Generic:Conn_02x03_Odd_Even
- added J6: P2, Connector_PinHeader_2.54mm:PinHeader_1x06_P2.54mm_Vertical, symbol Connector:Conn_01x06_Pin
- added JP1: SolderJumper_2_Open, Jumper:SolderJumper-2_P1.3mm_Open_RoundedPad1.0x1.5mm, symbol Jumper:SolderJumper_2_Open
- added LOGO1: Logo_Open_Hardware_Large, Symbol:OSHW-Logo_11.4x12mm_SilkScreen, symbol Graphic:Logo_Open_Hardware_Large
- added R1, R2: 22R, Resistor_SMD:R_0805_2012Metric, symbol Device:R
- added R3: 1M, Resistor_SMD:R_0805_2012Metric, symbol Device:R
- added R4: 10K, Resistor_SMD:R_0805_2012Metric, symbol Device:R
- added R5, R6, R7: 1K, Resistor_SMD:R_0805_2012Metric, symbol Device:R
- added TP2, TP3, TP4, TP5, TP6, TP8, TP9: TestPoint, TestPoint:TestPoint_Pad_D1.0mm, symbol Connector:TestPoint
- added U1: ATmega8U2-AU, Package_QFP:TQFP-32_7x7mm_P0.8mm, symbol MCU_Microchip_ATmega:ATmega8U2-A
- added VR1, VR2: CG0603MLC-05E, Resistor_SMD:R_0603_1608Metric, symbol Device:Varistor
- added Y1: 16MHz, Crystal:Crystal_SMD_Abracon_ABM3-2Pin_5.0x3.2mm, symbol Device:Crystal
Connections:
- new net: C3.1, R3.1, TP6.1, U1.1 (XTAL1), Y1.1
- new net: J6.2 (Pin_2), U1.12 (PD6)
- new net: J4.1 (Pin_1), U1.18 (PB4)
- new net: J4.3 (Pin_3), U1.19 (PB5)
- new net: C4.1, R3.2, TP8.1, U1.2 (PC0/XTAL2), Y1.2
- new net: J4.2 (Pin_2), U1.20 (PB6)
- new net: J4.4 (Pin_4), U1.21 (PB7)
- new net: J3.1 (Pin_1), U1.22 (PC7)
- new net: J3.2 (Pin_2), U1.23 (PC6)
- new net: J3.3 (Pin_3), U1.25 (PC5)
- new net: J3.4 (Pin_4), U1.26 (PC4)
- new net: C5.1, U1.27 (UCAP)
- new net: R1.1, U1.29 (D+)
- new net: R2.1, TP9.1, U1.30 (D-)
- new net: J3.5 (Pin_5), U1.5 (PC2)
- new net: J6.6 (Pin_6), U1.6 (PD0)
- new net: J6.5 (Pin_5), U1.7 (PD1)
- new net: J6.4 (Pin_4), U1.8 (PD2)
- new net: J6.3 (Pin_3), U1.9 (PD3)
- new net: J2.2 (D-), R2.2, VR2.1
- new net: FB1.1, J2.5 (Shield), VR1.2, VR2.2
- new net: J2.3 (D+), R1.2, TP5.1, VR1.1
- new net: F1.2, J2.1 (VBUS), TP3.1
- new net: D3.2 (A), R7.2
- new net: D2.2 (A), R6.2
- new net: C8.2, J6.1 (Pin_1)
- new net +5V: C1.1, C2.1, C7.1, D1.1 (K), J1.2, J1.3, J5.2 (Pin_2), R4.1, R6.1, R7.1, U1.32 (AVCC), U1.4 (VCC)
- new net DTR: C8.1, R5.1, U1.13 (~{HWB}/PD7)
- new net Earth: C5.2, C6.2, FB1.2, J2.4 (GND), JP1.1 (A), TP4.1, U1.28 (UGND)
- new net GND: C1.2, C2.2, C3.2, C4.2, C7.2, J1.1, J5.6 (Pin_6), JP1.2 (B), R5.2, U1.3 (GND)
- new net MISO2: J5.1 (Pin_1), U1.17 (PB3)
- new net MOSI2: J5.4 (Pin_4), U1.16 (PB2)
- new net RESET2: D1.2 (A), J5.5 (Pin_5), R4.2, U1.24 (PC1/~{RESET})
- new net RXLED: D2.1 (K), U1.10 (PD4)
- new net SCK2: J5.3 (Pin_3), U1.15 (PB1)
- new net TXLED: D3.1 (K), U1.11 (PD5)
- new net VBUS: C6.1, F1.1, TP2.1, U1.31 (UVCC)
- no-connect marks 0 -> 1
Other:
- note added: "KiBot variants example Not a real life board"
- note added: "Open source hardware"
- note added: "This logo has a REF starting with # Won't be passed to the PCB"
- note removed: "AN5346"
- note removed: "J. Pieper ADC investigation"
- note removed: "STM32G474 Datasheet p.81"
